Commit message: collision meshes updated

File: arm/arm_description/urdf/arm.urdf.xacro (robot description, xacro)
@@ -19,5 +19,5 @@
           <box size="0.0904 0.0901 0.08"/>
         </geometry>
-        <origin rpy="0 0 0" xyz="0 0 0"/>
+        <origin rpy="0 0 0" xyz="0 0 0.01"/>
       </collision>
       <inertial>
@@ -65,7 +65,7 @@
       <collision>
         <geometry>
-            <box size="0.056 0.0556 0.0207"/>
-          </geometry>
-        <origin rpy="0 0 0" xyz="0 0 0"/>
+            <box size="0.056 0.0556 0.005"/>
+          </geometry>
+        <origin rpy="0 0 0" xyz="0 0 -0.005"/>
       </collision>
       <inertial>
@@ -90,5 +90,5 @@
             <box size="0.05 0.032 0.04"/>
           </geometry>
-        <origin rpy="0 0 0" xyz="0 0 0"/>
+        <origin rpy="0 0 0" xyz="0.015 0 0"/>
       </collision>
       <inertial>
@@ -123,7 +123,7 @@
       <collision>
         <geometry>
-              <box size="0.048 0.0916 0.0286"/>
-          </geometry>
-        <origin rpy="0 0 0" xyz="0 0 0"/>
+              <box size="0.048 0.0550 0.0286"/>
+          </geometry>
+        <origin rpy="0 0 0" xyz="-0.0035 -0.010 0"/>
       </collision>
       <inertial>
@@ -148,5 +148,5 @@
             <box size="0.05 0.032 0.04"/>
           </geometry>
-        <origin rpy="0 0 0" xyz="0 0 0"/>
+        <origin rpy="0 0 0" xyz="0.015 0 0"/>
       </collision>
       <inertial>
@@ -181,7 +181,7 @@
       <collision>
         <geometry>
-             <box size="0.048 0.0916 0.0286"/>
-          </geometry>
-        <origin rpy="0 0 0" xyz="0 0 0"/>
+            <box size="0.048 0.0550 0.0286"/>
+          </geometry>
+        <origin rpy="0 0 0" xyz="-0.0035 -0.010 0"/>
       </collision>
       <inertial>
@@ -206,5 +206,5 @@
             <box size="0.05 0.032 0.04"/>
           </geometry>
-        <origin rpy="0 0 0" xyz="0 0 0"/>
+        <origin rpy="0 0 0" xyz="0.015 0 0"/>
       </collision>
       <inertial>
@@ -239,7 +239,7 @@
       <collision>
         <geometry>
-            <box size="0.0482 0.0547 0.043"/>
-        </geometry>
-        <origin rpy="0 0 0" xyz="0 0 0"/>
+            <box size="0.0482 0.0547 0.020"/>
+        </geometry>
+        <origin rpy="0 0 0" xyz="0.004 0 0.0025"/>
       </collision>
       <inertial>
@@ -262,7 +262,7 @@
       <collision>
         <geometry>
-           <box size="0.05 0.032 0.04"/>
-          </geometry>
-        <origin rpy="0 0 0" xyz="0 0 0"/>
+           <box size="0.05 0.032 0.035"/>
+          </geometry>
+        <origin rpy="0 0 0" xyz="0.015 0 0.0001"/>
       </collision>
       <inertial>
@@ -299,5 +299,5 @@
               <box size="0.1044 0.0578 0.005"/>
           </geometry>
-        <origin rpy="0 0 0" xyz="0 0 0"/>
+        <origin rpy="0 0 0" xyz="0 0 0.0005"/>
       </collision>
       <inertial>
@@ -325,5 +325,5 @@
              <box size="0.0629 0.0312 0.0408"/>
           </geometry>
-        <origin rpy="0 0 0" xyz="0 0 0"/>
+        <origin rpy="0 0 0" xyz="0.025 0 0"/>
       </collision>
       <inertial>
@@ -351,5 +351,5 @@
              <box size="0.0629 0.0312 0.0408"/>
           </geometry>
-        <origin rpy="0 0 0" xyz="0 0 0"/>
+        <origin rpy="0 0 0" xyz="0.025 0 0"/>
       </collision>
       <inertial>
