Commit message: collision meshes updated

File: arm/arm_description/urdf/camera.xacro (robot description, xacro)
@@ -14,5 +14,5 @@
          <box size="0.0225 0.0225 0.0225"/>
         </geometry>
-        <origin rpy="0 0 0" xyz="0 0 0"/>
+        <origin rpy="0 0 0" xyz="0 0 -0.02"/>
       </visual>
       <collision>
@@ -20,5 +20,5 @@
             <box size="0.0225 0.0225 0.0225"/>
           </geometry>
-        <origin rpy="0 0 0" xyz="0 0 0"/>
+        <origin rpy="0 0 0" xyz="0 0 -0.02"/>
       </collision>
     </link>
